File: KiCadSchematics/TachometerProject/KeypadReader.kicad_sch (KiCad schematic)
At the start: 12 parts

Commit message: Updated circuit diagrams
Connections:
- net at R?.1, R?.1, R?.2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: now also U?.18 (B.0); no longer U?.19 (A.0)
Changed lines of the file:
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@@
+    (stroke (width 0) (type default) (color 0 0 0 0))
+  )
+  (wire (pts (xy 161.29 81.28) (xy 168.91 81.28))
     (stroke (width 0) (type default) (color 0 0 0 0))
   )
@@
     (stroke (width 0) (type default) (color 0 0 0 0))
   )
-  (wire (pts (xy 168.91 118.11) (xy 168.91 78.74))
+  (wire (pts (xy 168.91 118.11) (xy 168.91 81.28))
     (stroke (width 0) (type default) (color 0 0 0 0))
   )
@@
     (stroke (width 0) (type default) (color 0 0 0 0))
   )
-  (wire (pts (xy 168.91 78.74) (xy 161.29 78.74))
-    (stroke (width 0) (type default) (color 0 0 0 0))
-  )
