File: KiCadSchematics/TachometerProject/MeasurementDevice.kicad_sch (KiCad schematic)
At the start: 5 parts

Commit message: Exported and Added SVG drawings
Parts:
- gave numbers to parts that had none: 2
Changed lines of the file:
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@@
   (symbol (lib_id "Device:R_US") (at 88.9 60.96 0) (unit 1)
     (in_bom yes) (on_board yes) (fields_autoplaced)
-    (property "Reference" "R?" (id 0) (at 91.44 59.6899 0)
+    (property "Reference" "R1" (id 0) (at 91.44 59.6899 0)
       (effects (font (size 1.27 1.27)) (justify left))
     )
@@
   (symbol (lib_id "Device:R_US") (at 105.41 39.37 0) (unit 1)
     (in_bom yes) (on_board yes) (fields_autoplaced)
-    (property "Reference" "R?" (id 0) (at 107.95 38.0999 0)
+    (property "Reference" "R2" (id 0) (at 107.95 38.0999 0)
       (effects (font (size 1.27 1.27)) (justify left))
     )

Commit message: Updated Schematic Drawings, README
Connections:
- net OMD Output: now reaches U?.3 (Output)
Changed lines of the file:
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@@
+    (stroke (width 0) (type default) (color 0 0 0 0))
+  )
+  (wire (pts (xy 116.84 71.12) (xy 121.92 71.12))
+    (stroke (width 0) (type default) (color 0 0 0 0))
+  )
+  (wire (pts (xy 128.27 49.53) (xy 116.84 49.53))
     (stroke (width 0) (type default) (color 0 0 0 0))
   )
@@
   )
   (wire (pts (xy 162.56 49.53) (xy 153.67 49.53))
+    (stroke (width 0) (type default) (color 0 0 0 0))
+  )
+  (wire (pts (xy 116.84 49.53) (xy 116.84 71.12))
     (stroke (width 0) (type default) (color 0 0 0 0))
   )
@@
     (effects (font (size 1.27 1.27)) (justify left bottom))
   )
+  (hierarchical_label "OMD Output" (shape input) (at 121.92 71.12 0)
+    (effects (font (size 1.27 1.27)) (justify left))
+  )
   (symbol (lib_id "power:Earth") (at 105.41 64.77 0) (unit 1)

Commit message: Updated circuit diagrams
Changed lines of the file:
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@@
     (effects (font (size 1.27 1.27)) (justify left bottom))
   )
-  (hierarchical_label "OMD Output" (shape input) (at 121.92 71.12 0)
+  (hierarchical_label "OMD Output" (shape output) (at 121.92 71.12 0)
     (effects (font (size 1.27 1.27)) (justify left))
   )

Commit message: Schematic update
Parts:
- R1: value 50Ω -> 51Ω
Changed lines of the file:
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@@
       (effects (font (size 1.27 1.27)) (justify left))
     )
-    (property "Value" "50Ω" (id 1) (at 91.44 62.2299 0)
+    (property "Value" "51Ω" (id 1) (at 91.44 62.2299 0)
       (effects (font (size 1.27 1.27)) (justify left))
     )
