File: KiCadSchematics/TachometerProject/TachometerProject.kicad_sch (KiCad schematic)
At the start: 0 parts

Commit message: Exported and Added SVG drawings
Parts:
- added U?: Level_Shifter, symbol EGR_270:Level_Shifter
- added U?: RaspberryPiConnector, symbol EGR_270:RaspberryPiConnector
Connections:
- new net: U?.1 (LV1), U?.2 (SDA1)
- new net: U?.2 (LV2), U?.3 (SCL1)
- new net: U?.1 (3V3), U?.3 (LV)
- new net: U?.4 (GND), U?.5 (GND)
- new net +5V: U?.10 (HV)
- new net Earth: U?.9 (GND)
Other:
- added sheet FrequencyDivider (FrequencyDivider.kicad_sch)

Commit message: Updated Schematic Drawings, README
Connections:
- net LCD SCL: now reaches U?.11 (HV2)
- net LCD SDA: now reaches U?.12 (HV1)
- net at U?.5 (LV3): now also U?.6 (GPIO17)
- net FrequencyDivider/RPi PWM: now reaches U?.8 (HV3)
Other:
- sheet FrequencyDivider ports: added OMD Output, RPi PWM, SCL, SDA, Strobe Trigger; removed none
- sheet KeypadReader ports: added SCL, SDA; removed none
- sheet OpticalMeasurementDevice ports: added OMD Output; removed none
- sheet Strobing Circuit ports: added Strobe Trigger; removed none

Commit message: Updated circuit diagrams
Connections:
- net FrequencyDivider/OMD Output: now also U?.7 (HV4)
- net at U?.6 (LV4): now also U?.7 (GPIO27)
